File: Hardware Files/HotPlateController.kicad_pcb (KiCad board)
At the start: 2 copper layers, 14 parts, among them J1 Thermocouple, J2 Screw_Terminal_01x03, J3 Screw_Terminal_01x03, J5 0.100" 2x4 Header, SW1 SPST (BLUE), SW2 SPST (RED), U1 ESP32-WROOM-32, U2 ACS712xLCTR-20A, U3 MAX31855KASA

Commit message: Fix footprints
Parts:
- removed D1, D2: LED, Diode_SMD:D_1206_3216Metric_Pad1.42x1.75mm_HandSolder
- removed J1: Thermocouple, TerminalBlock_TE-Connectivity:TerminalBlock_TE_282834-2_1x02_P2.54mm_Horizontal
- removed J2, J3: Screw_Terminal_01x03, TerminalBlock:TerminalBlock_bornier-3_P5.08mm
- removed J5: 0.100" 2x4 Header, Connector_PinHeader_2.54mm:PinHeader_2x04_P2.54mm_Vertical
- removed PS1: HLK-PM01, Converter_ACDC:Converter_ACDC_HiLink_HLK-PMxx
- removed R1, R2: R, Resistor_SMD:R_1206_3216Metric_Pad1.30x1.75mm_HandSolder
- removed SW1: SPST (BLUE), .DesignArchive:PTS636_SM25F_SMTR_LFS
- removed SW2: SPST (RED), .DesignArchive:PTS636_SM25F_SMTR_LFS
- removed U1: ESP32-WROOM-32, RF_Module:ESP32-WROOM-32
- removed U2: ACS712xLCTR-20A, Package_SO:SOIC-8_3.9x4.9mm_P1.27mm
- removed U3: MAX31855KASA, Package_SO:SOIC-8_3.9x4.9mm_P1.27mm

Commit message: Add Relay level shifter
Parts:
- added C1: 220nF 50V, Capacitor_SMD:C_1206_3216Metric_Pad1.33x1.80mm_HandSolder, F.Cu at (144.2, 23.3)
- added C2: 220nF 50V, Capacitor_SMD:C_1206_3216Metric_Pad1.33x1.80mm_HandSolder, F.Cu at (144.2, 20.0)
- added C3: 10uF 25V 10%, Capacitor_SMD:C_1206_3216Metric, F.Cu at (205.0, 10.0)
- added C4: 1uF 50V, Capacitor_SMD:C_1206_3216Metric, F.Cu at (205.0, 13.3)
- added C5: 1uF 50V, Capacitor_SMD:C_1206_3216Metric, F.Cu at (210.7, 10.0)
- added C6: 1nF 50V, Capacitor_SMD:C_1206_3216Metric, F.Cu at (205.0, 16.7)
- added C7: 1nF 50V, Capacitor_SMD:C_1206_3216Metric, F.Cu at (210.7, 13.3)
- added C8: 1nF 50V, Capacitor_SMD:C_1206_3216Metric, F.Cu at (216.3, 10.0)
- added D1: LED, Capacitor_SMD:C_1206_3216Metric, F.Cu at (192.9, 11.0)
- added D2: LED, Capacitor_SMD:C_1206_3216Metric, F.Cu at (192.9, 7.65)
- added J1: 0.100" 2x4 Header, Connector_PinHeader_2.54mm:PinHeader_2x04_P2.54mm_Vertical, F.Cu at (143.5, 8.38)
- added J2: Screw_Terminal_01x03, TerminalBlock:TerminalBlock_bornier-3_P5.08mm, F.Cu at (136.0, 50.0)
- added J3: Screw_Terminal_01x03, TerminalBlock:TerminalBlock_bornier-3_P5.08mm, F.Cu at (254.0, 60.0)
- added J4: Conn_01x02, HotPlateController:1935161, F.Cu at (135.0, 104.0)
- added J5: Thermocouple, HotPlateController:1935161, F.Cu at (136.0, 139.0)
- added PS1: HLK-PM01, Converter_ACDC:Converter_ACDC_HiLink_HLK-PMxx, F.Cu at (180.0, 50.0)
- added R1: 1.37k 0.25W 1%, Resistor_SMD:R_1206_3216Metric, F.Cu at (210.6, 16.7)
- added R2: 2.67k 0.25W 1%, Resistor_SMD:R_1206_3216Metric, F.Cu at (216.3, 13.3)
- added R3: 10k 5% 0.25W, Resistor_SMD:R_1206_3216Metric, F.Cu at (221.9, 9.97)
- added R4: 10k 5% 0.25W, Resistor_SMD:R_1206_3216Metric, F.Cu at (216.2, 16.7)
- added R5: R, Resistor_SMD:R_1206_3216Metric, F.Cu at (192.8, 14.4)
- added R6: 10k 5% 0.25W, Resistor_SMD:R_1206_3216Metric, F.Cu at (221.9, 13.3)
- added R7: R, Resistor_SMD:R_1206_3216Metric, F.Cu at (192.8, 17.7)
- added SW1: SPST (BLUE), .DesignArchive:PTS636_SM25F_SMTR_LFS, F.Cu at (150.1, 13.3)
- added SW2: SPST (RED), .DesignArchive:PTS636_SM25F_SMTR_LFS, F.Cu at (150.1, 8.46)
- added U1: NCP1117ST33T3G, Package_TO_SOT_SMD:SOT-223-3_TabPin2, F.Cu at (153.3, 19.8)
- added U2: ACS712xLCTR-20A, Package_SO:SOIC-8_3.9x4.9mm_P1.27mm, F.Cu at (194.1, 2.73)
- added U3: ESP32-WROOM-32, RF_Module:ESP32-WROOM-32, F.Cu at (228.0, 131.0)
- added U4: MAX31855KASA, Package_SO:SOIC-8_3.9x4.9mm_P1.27mm, F.Cu at (160.0, 139.0)

Commit message: Begin Layout
Parts:
- removed the J4 at (135.0, 104.0)
- added J1: Conn_01x02, HotPlateController:1935161, F.Cu at (136.0, 85.0)
- added Q1: NMOS 60V 300mA, Package_TO_SOT_SMD:SOT-23, F.Cu at (139.0, 96.0)
- added Q2: NMOS 60V 46A, Package_TO_SOT_SMD:TO-252-3_TabPin2, F.Cu at (146.0, 93.0)
- added R1: 10k 5% 0.25W, Resistor_SMD:R_1206_3216Metric, F.Cu at (146.0, 101.0)
- moved C2 157.4 mm to (247.2, 139.0)
- moved J2 157.4 mm to (246.5, 127.4)
- moved SW1 157.4 mm to (253.1, 132.3)
- moved SW2 157.4 mm to (253.1, 127.5)
- moved C1 157.4 mm to (247.2, 142.3)
- moved U1 69.2 mm to (203.0, 68.0), turned to 270 degrees
- moved U2 67.6 mm to (246.0, 46.0), turned to 90 degrees
- moved C6 48.0 mm to (247.5, 39.0), turned to 90 degrees
- moved C5 46.7 mm to (241.5, 45.0), turned to 90 degrees
- moved R2 41.0 mm to (245.0, 39.0), turned to 90 degrees
- moved R3 36.7 mm to (242.5, 39.0), turned to 270 degrees
- renumbered J1 to J2, J2 to J3, J3 to J4, J5 to J6, R1 to R2, R2 to R3, R3 to R4, R4 to R5, R5 to R6, R6 to R7, R7 to R8

Commit message: add 3 pos terminal footprint
Parts:
- added M1: Conn_01x01, MountingHole:MountingHole_3.2mm_M3_DIN965, F.Cu at (5.00, 5.00)
- added M2: Conn_01x01, MountingHole:MountingHole_3.2mm_M3_DIN965, F.Cu at (5.00, 70.0)
- added M3: Conn_01x01, MountingHole:MountingHole_3.2mm_M3_DIN965, F.Cu at (70.0, 5.00)
- added M4: Conn_01x01, MountingHole:MountingHole_3.2mm_M3_DIN965, F.Cu at (70.0, 70.0)
- moved C1 237.5 mm to (34.0, 37.6), turned to 270 degrees
- moved C2 229.5 mm to (37.5, 45.5), turned to 180 degrees
- moved J2 203.6 mm to (64.0, 37.0)
- moved SW2 202.1 mm to (63.0, 58.8), turned to 90 degrees
- moved U3 201.3 mm to (40.0, 59.0), turned to 180 degrees
- moved SW1 200.1 mm to (67.0, 58.8), turned to 90 degrees
- moved R7 198.9 mm to (26.5, 50.5), turned to 180 degrees
- moved C6 195.8 mm to (52.5, 21.0), turned to 270 degrees
- moved U2 194.6 mm to (54.0, 14.0), turned to 270 degrees
- moved J4 191.6 mm to (66.0, 23.0)
- moved R2 190.9 mm to (55.0, 21.0), turned to 270 degrees
- moved R3 185.9 mm to (57.5, 21.0), turned to 90 degrees
- moved C5 185.4 mm to (58.5, 15.0), turned to 270 degrees
- moved R4 169.5 mm to (57.5, 51.0)
- moved U4 167.0 mm to (17.5, 52.0)
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Connections:
- U2 pad 1: Net-(J3-Pad1) -> Net-(J4-Pad3)
- U2 pad 2: Net-(J3-Pad1) -> Net-(J4-Pad3)
- U2 pad 3: Net-(J4-Pad3) -> Net-(J3-Pad1)
- U2 pad 4: Net-(J4-Pad3) -> Net-(J3-Pad1)
- U3 pad 2: Net-(U3-Pad2) -> +3V3
- U3 pad 23: Net-(U3-Pad23) -> U0TX_Active
Other:
- board outline added: 75 x 75 mm
- board text added: "E|N|L"
- board text added: "L|N|E"

Commit message: Bulk routing
Parts:
- added C9: 1uF 50V, Capacitor_SMD:C_1206_3216Metric, F.Cu at (17.5, 56.4)
- D1, D2: footprint Capacitor_SMD:C_1206_3216Metric -> Diode_SMD:D_1206_3216Metric_Pad1.42x1.75mm_HandSolder
- J3, J4: footprint TerminalBlock:TerminalBlock_bornier-3_P5.08mm -> HotPlateController:1729131
- PS1: footprint Converter_ACDC:Converter_ACDC_HiLink_HLK-PMxx -> HotPlateController:Converter_ACDC_HiLink_HLK-PMxx
- SW1, SW2: footprint .DesignArchive:PTS636_SM25F_SMTR_LFS -> HotPlateController:PTS636_SM25F_SMTR_LFS
- moved C5 15.9 mm to (60.5, 30.7), turned to 90 degrees
- moved R2 14.3 mm to (65.5, 30.7), turned to 90 degrees
- moved U2 14.0 mm to (55.6, 27.9)
- moved C6 12.3 mm to (53.1, 33.3), turned to 180 degrees
- moved C1 11.7 mm to (45.7, 38.1), turned to 90 degrees
- moved R3 11.2 mm to (63.0, 30.7), turned to 270 degrees
- moved C2 8.65 mm to (33.0, 38.1), turned to 270 degrees
- moved SW2 7.87 mm to (70.9, 58.4)
- moved D1 5.59 mm to (59.5, 40.0)
- moved R6 5.59 mm to (59.5, 37.5)
- moved J2 4.00 mm to (68.0, 37.0)
- moved D2 3.64 mm to (51.5, 40.0)
- moved R8 3.64 mm to (51.5, 37.5)
- moved C7 1.46 mm to (59.0, 58.5)
- moved C8 1.46 mm to (59.0, 53.5)
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Connections:
- U3 pad 19: Net-(U3-Pad19) -> /ESP32_SPI_MISO
- U3 pad 37: Net-(U3-Pad37) -> /ESP32_SPI_TEMPSENSOR_1_CS
- U3 pad 5: Net-(U3-Pad5) -> /ESP32_SPI_SCK
Routing:
- net +3V3: track 0.00 -> 107.9 mm, vias 0 -> 2
- net +5V: track 0.00 -> 83.7 mm
- net UserSwitch: track 0.00 -> 77.9 mm, vias 0 -> 3
- net /USB_TX: track 0.00 -> 67.6 mm, vias 0 -> 1
- net /EN: track 0.00 -> 67.3 mm, vias 0 -> 2
- net Net-(J3-Pad2): track 0.00 -> 61.1 mm
- net Earth: track 0.00 -> 59.9 mm
- net /USB_RX: track 0.00 -> 58.4 mm, vias 0 -> 1
- net V_Current_adj: track 0.00 -> 48.9 mm, vias 0 -> 2
- net Net-(J1-Pad1): track 0.00 -> 38.2 mm
- net /ESP32_SPI_SCK: track 0.00 -> 36.9 mm, vias 0 -> 2
- net /ESP32_SPI_MISO: track 0.00 -> 26.2 mm
- net /ESP32_SPI_TEMPSENSOR_1_CS: track 0.00 -> 22.1 mm
- net V_Current: track 0.00 -> 14.5 mm
- net U0TX_Active: track 0.00 -> 12.4 mm
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- added copper zone on B.Cu, net GND
- added copper zone on F.Cu, net GND
- added copper zone on F.Cu, net Net-(J3-Pad1)
- added copper zone on B.Cu, net Net-(J4-Pad3)
- added copper zone on F.Cu, net Net-(J4-Pad3)
- added copper zone on F.Cu, net Net-(J6-Pad1)
- added copper zone on F.Cu, net Net-(J6-Pad2)
Other:
- outline, holes or cut-outs redrawn
- board text removed: "E|N|L"
- board text removed: "L|N|E"

Commit message: Add artwork update PCBA Rev Silkscreen
Parts:
- added G***: LOGO, MicroBBPS:PCBA Revision, F.Cu at (15.0, 64.5)
- added G***: LOGO, 8Bit_WiFi_Visualizer_Footprints:logo, F.Cu at (14.0, 60.5)
- added G***: LOGO, HotPlateController:test2, B.Cu at (37.5, 37.5)

Commit message: Update Part Ordering Information
Parts:
- removed G***: LOGO, MicroBBPS:PCBA Revision
- removed G***: LOGO, 8Bit_WiFi_Visualizer_Footprints:logo
- removed G***: LOGO, HotPlateController:test2
- added R9: 0R, Resistor_SMD:R_2512_6332Metric_Pad1.40x3.35mm_HandSolder, F.Cu at (56.4, 12.7)
- D1: value LED -> Green 3.0V
- D2: value LED -> Orange 2.0V
- J6: value Thermocouple -> Conn_01x02
- Q2: value NMOS 60V 46A -> NMOS 60V 3A
- R6: value R -> 0R
- R8: value R -> 43.2R
- SW1: value SPST (BLUE) -> SPST
- SW2: value SPST (RED) -> SPST
Connections:
- U3 pad 16: Net-(U3-Pad16) -> StatusLED
- U3 pad 17: Net-(U3-Pad17) -> HotLED
Routing:
- net StatusLED: track 0.00 -> 19.7 mm, vias 0 -> 2
- net HotLED: track 0.00 -> 13.5 mm, vias 0 -> 2

Commit message: Finalize board layout and art
Parts:
- added G***: LOGO, HotPlateController:test2, B.Cu at (37.5, 37.5)
- added G***: LOGO, HotPlateController:silkscreenart, F.Cu at (39.1, 34.7)
