File: Hardware Files/HotPlateController.kicad_pcb (KiCad board)
At the start: 2 copper layers, 75 x 75 mm, 40 parts, among them J1 Conn_01x02, J2 0.100" 2x4 Header, J3 Screw_Terminal_01x03, J4 Screw_Terminal_01x03, J6 Conn_01x02, M1 Conn_01x01, M2 Conn_01x01, M3 Conn_01x01, M4 Conn_01x01, Q1 NMOS 60V 300mA, Q2 NMOS 60V 3A, SW1 SPST, SW2 SPST, U1 NCP1117ST33T3G, U2 ACS712xLCTR-20A, U3 ESP32-WROOM-32, U4 MAX31855KASA

Commit message: Finalize A01 Design
Connections:
- J2 pad 7: /VREG_IN -> +5V
Routing:
- net +5V: track 83.7 -> 105.9 mm, vias 0 -> 1
